File: hardware/voice/AS3397_proto_SMS.kicad_sch (KiCad schematic)
At the start: 105 parts, among them J1 ES, Q1 BS170F, Q2 BS170F, Q3 BS170F, Q4 BS170F, Q5 BS170F, U1 MCP6002, U2 Pico, U3 MCP6002, U4 MCP6002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

Commit message: Better documentation
Other:
- note added: "16 bits PWM"
- note added: "3.3V -> 5V level shifter PWM low-pass filtering"
- note added: "AS3397"
- note added: "Audio output (transimpedance opAmp)"
- note added: "DCO charge condensator DCO ramp to ADC"
- note added: "External Power pins"
- note added: "Pi pico (rp2040)"
- note added: "Registers change"
- note added: "Wave Select"
- moved on the sheet: AS1, C1, C10, C11, C12, C13, C14, C15, C16, C17, C18, C19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

Commit message: Draft Article without todo list in french
Other:
- note added: "3.3V -> 5V"
- note added: "Filter CutOff Control Voltage"
- note added: "Pulse Width Control Voltage"
- note added: "level shifter PWM low-pass filtering"
- note removed: "3.3V -> 5V level shifter PWM low-pass filtering"
- moved on the sheet: C31, C32, C35, C36, R39, R40, R41, R42, R43, R44, R45, R46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

Commit message: DCO documentation - Waveshapper, Square wave
Parts:
- R20: value 33k -> 27k
Changed lines of the file:
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@@
       (effects (font (size 1.27 1.27)))
     )
-    (property "Value" "33k" (at 162.56 311.15 90)
+    (property "Value" "27k" (at 162.56 311.15 90)
       (effects (font (size 1.27 1.27)))
     )
