File: hardware/voice/eurorack-smd-0603/AS3397_eurorack_0603.kicad_pcb (KiCad board)
At the start: 2 copper layers, 59.7 x 57.2 mm, 110 parts, among them J1 Conn_01x04_Socket_I2C, J2 Conn_01x03_Socket_Audio, J4 Conn_01x04_Socket_POWER, Q1 BS170F, Q2 BS170F, Q3 BS170F, Q4 BS170F, Q5 BS170F, U1 MCP6002, U2 Pico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

Commit message: Voice PCB directory cleanup bis
Parts:
- U2: footprint SYNTHFILLE:RPi_Pico_SMD_AS -> AS3397_eurorack_0603:RPi_Pico_SMD_TH
- moved Q1 4.53 mm to (188.7, 49.9)
- moved U2 2.21 mm to (189.5, 67.8)
Connections:
- U2 pad 1: (no net) -> PWM_3.3V_PAN_CV
- U2 pad 10: (no net) -> PWM_3.3V_FITLER_FREQ_CV
- U2 pad 11: (no net) -> GAMME_B
- U2 pad 12: (no net) -> PULSE_PIO_FREQ_B
- U2 pad 13: (no net) -> GND
- U2 pad 14: (no net) -> V_WF_A_MSB_PWM
- U2 pad 15: (no net) -> V_WF_A_LSB_PWM
- U2 pad 16: (no net) -> V_WF_B_MSB_PWM
- U2 pad 17: (no net) -> V_WF_B_LSB_PWM
- U2 pad 18: (no net) -> GND
- U2 pad 19: (no net) -> DSO_MSB_PWM
- U2 pad 2: (no net) -> PWM_3.3V_MOD_AMOUNT_CV
- U2 pad 20: (no net) -> DSO_LSB_PWM
- U2 pad 21: (no net) -> WS_BIT0
- U2 pad 22: (no net) -> unconnected-(U2-GPIO17-Pad22)
- U2 pad 23: (no net) -> GND
- U2 pad 24: (no net) -> GAMME_A
- U2 pad 25: (no net) -> PULSE_PIO_FREQ_A
- U2 pad 26: (no net) -> I2C_SDA
- U2 pad 27: (no net) -> I2C_SCK
- U2 pad 28: (no net) -> GND
- U2 pad 29: (no net) -> WS_BIT1
- U2 pad 3: (no net) -> GND
- U2 pad 30: (no net) -> unconnected-(U2-RUN-Pad30)
- U2 pad 31: (no net) -> ADC_0
- U2 pad 32: (no net) -> ADC_1
- U2 pad 33: (no net) -> GND
- U2 pad 34: (no net) -> I2C_ADR
- U2 pad 35: (no net) -> unconnected-(U2-ADC_VREF-Pad35)
- U2 pad 36: (no net) -> +3.3V
- U2 pad 37: (no net) -> unconnected-(U2-3V3_EN-Pad37)
- U2 pad 38: (no net) -> GND
- U2 pad 39: (no net) -> VBUS
- U2 pad 4: (no net) -> PWM_3.3V_PULSE_WIDTH_A_C.V
- U2 pad 40: (no net) -> Net-(Q1-G)
- U2 pad 5: (no net) -> PWM_3.3V_PULSE_WIDTH_B_C.V
- U2 pad 6: (no net) -> PWM_3.3V_BALANCE_CV
- U2 pad 7: (no net) -> PWM_3.3V_LINEAR_GAIN_CV
- U2 pad 8: (no net) -> GND
- U2 pad 9: (no net) -> PWM_3.3V_RESONANCE_CV

Commit message: Power board
Parts:
- moved C18 243.9 mm to (243.1, 56.2)
- moved C14 237.4 mm to (245.7, 59.9), turned to 90 degrees
- moved C19 237.3 mm to (237.9, 63.2)
- moved C13 232.6 mm to (233.5, 58.2), turned to 90 degrees
- moved U4 232.3 mm to (239.7, 59.7)
- moved R17 224.3 mm to (244.2, 59.8), turned to 90 degrees
- moved R16 221.9 mm to (235.1, 58.3), turned to 90 degrees
- moved C31 184.7 mm to (239.2, 76.7)
- moved C7 181.5 mm to (203.5, 74.3), turned to -90 degrees
- moved C28 180.9 mm to (278.4, 81.0)
- moved C29 180.7 mm to (272.0, 89.0)
- moved R4 180.5 mm to (201.2, 79.3)
- moved D2 180.4 mm to (267.9, 80.7)
- moved R3 180.4 mm to (201.1, 76.7)
- moved C32 178.7 mm to (233.3, 84.8), turned to -90 degrees
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Routing:
- net PWM_5V_PAN_CV: track 0.00 -> 80.8 mm
- net PWM_5V_LINEAR_GAIN_CV: track 0.00 -> 43.9 mm
- net V_WF_A: track 0.00 -> 41.8 mm, vias 0 -> 2
- net PWM_DAC_PULSE_WIDTH_A: track 0.00 -> 35.8 mm
- net CTA: track 0.00 -> 30.6 mm
- net PWM_DAC_PULSE_WIDTH_B: track 0.00 -> 28.4 mm
- net V_WF_B: track 0.00 -> 27.9 mm
- net PWM_5V_FITLER_FREQ_CV: track 0.00 -> 25.0 mm
- net PWM_3.3V_PAN_CV: track 0.00 -> 24.9 mm, vias 0 -> 1
- net CTB: track 5.17 -> 29.6 mm
- net PWM_3.3V_MOD_AMOUNT_CV: track 0.00 -> 24.1 mm, vias 0 -> 1
- net Output_VCA_R: track 0.00 -> 23.5 mm
- net PWM_5V_MOD_AMOUNT_CV: track 0.00 -> 14.7 mm, vias 0 -> 1
- net +5V: track 0.00 -> 13.1 mm
- net PWM_5V_BALANCE_CV: track 0.00 -> 10.3 mm
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Other:
- board size 59.7 x 57.2 mm -> 92.2 x 64.2 mm
