File: hardware/power/powerBoard.kicad_sch (KiCad schematic)
At the start: 19 parts, among them J1 Conn_01x03_Socket, J2 Conn_02x05_Odd_Even, U1 LM2575-5.0BT, U2 LM2575-5.0BT

Commit message: hardware readme
Parts:
- J1: value Conn_01x03_Socket -> 12V_screw_terminal
Other:
- moved on the sheet: C1, C2, C3, C4, D1, D2, D3, D4, D5, J1, J2, L1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
