File: hardware/voice/main-smd-1206/AS3397_proto_SMS.kicad_sch (KiCad schematic)
At the start: 105 parts, among them J1 ES, Q1 BS170F, Q2 BS170F, Q3 BS170F, Q4 BS170F, Q5 BS170F, U1 MCP6002, U2 Pico, U3 MCP6002, U4 MCP6002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

Commit message: Through hole voice board first commit
Parts:
- U1, U3, U5, U7: value MCP6002 -> TS922
Changed lines of the file:
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@@
       (effects (font (size 1.27 1.27)))
     )
-    (property "Value" "MCP6002" (at 365.76 229.87 0)
+    (property "Value" "TS922" (at 365.76 229.87 0)
       (effects (font (size 1.27 1.27)))
     )
@@
       (effects (font (size 1.27 1.27)))
     )
-    (property "Value" "MCP6002" (at 266.7 242.57 0)
+    (property "Value" "TS922" (at 266.7 242.57 0)
       (effects (font (size 1.27 1.27)))
     )
@@
       (effects (font (size 1.27 1.27)))
     )
-    (property "Value" "MCP6002" (at 412.75 334.01 0)
+    (property "Value" "TS922" (at 412.75 334.01 0)
       (effects (font (size 1.27 1.27)))
     )
@@
       (effects (font (size 1.27 1.27)))
     )
-    (property "Value" "MCP6002" (at 193.04 294.64 0)
+    (property "Value" "TS922" (at 193.04 294.64 0)
       (effects (font (size 1.27 1.27)))
     )
@@
       (effects (font (size 1.27 1.27)))
     )
-    (property "Value" "MCP6002" (at 365.76 180.34 0)
+    (property "Value" "TS922" (at 365.76 180.34 0)
       (effects (font (size 1.27 1.27)))
     )
@@
       (effects (font (size 1.27 1.27)))
     )
-    (property "Value" "MCP6002" (at 412.75 220.98 0)
+    (property "Value" "TS922" (at 412.75 220.98 0)
       (effects (font (size 1.27 1.27)))
     )
@@
       (effects (font (size 1.27 1.27)))
     )
-    (property "Value" "MCP6002" (at 215.9 223.52 0)
+    (property "Value" "TS922" (at 215.9 223.52 0)
       (effects (font (size 1.27 1.27)))
     )
@@
       (effects (font (size 1.27 1.27)))
     )
-    (property "Value" "MCP6002" (at 363.22 353.06 0)
+    (property "Value" "TS922" (at 363.22 353.06 0)
       (effects (font (size 1.27 1.27)))
     )
@@
       (effects (font (size 1.27 1.27)))
     )
-    (property "Value" "MCP6002" (at 215.9 328.93 0)
+    (property "Value" "TS922" (at 215.9 328.93 0)
       (effects (font (size 1.27 1.27)))
     )
@@
       (effects (font (size 1.27 1.27)))
     )
-    (property "Value" "MCP6002" (at 215.9 254 0)
+    (property "Value" "TS922" (at 215.9 254 0)
       (effects (font (size 1.27 1.27)))
     )
@@
       (effects (font (size 1.27 1.27)))
     )
-    (property "Value" "MCP6002" (at 77.47 208.28 0)
+    (property "Value" "TS922" (at 77.47 208.28 0)
       (effects (font (size 1.27 1.27)))
     )
@@
       (effects (font (size 1.27 1.27)))
     )
-    (property "Value" "MCP6002" (at 363.22 300.99 0)
+    (property "Value" "TS922" (at 363.22 300.99 0)
       (effects (font (size 1.27 1.27)))
     )
