File: hardware/voice/main-smd-1206/AS3397_proto_SMS.kicad_pcb (KiCad board)
At the start: 2 copper layers, 71.1 x 104.1 mm, 105 parts, among them J1 ES, Q1 BS170F, Q2 BS170F, Q3 BS170F, Q4 BS170F, Q5 BS170F, U1 MCP6002, U2 Pico, U3 MCP6002, U4 MCP6002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

Commit message: Voice PCB directory cleanup
Parts:
- R20: value 33k -> 27k
- U2: footprint SYNTHFILLE:RPi_Pico_SMD_AS -> AS3397_proto_SMS:RPi_Pico_SMD_TH
Changed lines of the file:
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@@
     )
   )
-  (footprint "SYNTHFILLE:RPi_Pico_SMD_AS" (layer "F.Cu")
+  (footprint "AS3397_proto_SMS:RPi_Pico_SMD_TH" (layer "F.Cu")
     (at 123.444 110.363)
     (descr "Through hole straight pin header, 2x20, 2.54mm pitch, double rows")
@@
     (property "Sheetname" "")
     (attr through_hole)
-    (fp_text reference "U2" (at -2.54 1.905) (layer "F.SilkS")
-        (effects (font (size 1 1) (thickness 0.15)))
-    )
-    (fp_text value "Pico" (at -5.461 6.604) (layer "F.Fab")
+    (fp_text reference "U2" (at 0 0) (layer "F.SilkS")
+        (effects (font (size 1 1) (thickness 0.15)))
+    )
+    (fp_text value "Pico" (at 0 2.159) (layer "F.Fab")
+        (effects (font (size 1 1) (thickness 0.15)))
+    )
+    (fp_text user "GP1" (at -12.9 -21.6 45) (layer "F.SilkS")
+        (effects (font (size 0.8 0.8) (thickness 0.15)))
+    )
+    (fp_text user "GP4" (at -12.8 -11.43 45) (layer "F.SilkS")
+        (effects (font (size 0.8 0.8) (thickness 0.15)))
+    )
+    (fp_text user "GND" (at 12.8 6.35 45) (layer "F.SilkS")
+        (effects (font (size 0.8 0.8) (thickness 0.15)))
+    )
+    (fp_text user "GND" (at -12.8 19.05 45) (layer "F.SilkS")
+        (effects (font (size 0.8 0.8) (thickness 0.15)))
+    )
+    (fp_text user "GP10" (at -13.054 8.89 45) (layer "F.SilkS")
+        (effects (font (size 0.8 0.8) (thickness 0.15)))
+    )
+    (fp_text user "VSYS" (at 13.2 -21.59 45) (layer "F.SilkS")
+        (effects (font (size 0.8 0.8) (thickness 0.15)))
+    )
+    (fp_text user "GP13" (at -13.054 16.51 45) (layer "F.SilkS")
+        (effects (font (size 0.8 0.8) (thickness 0.15)))
+    )
+    (fp_text user "3V3" (at 12.9 -13.9 45) (layer "F.SilkS")
+        (effects (font (size 0.8 0.8) (thickness 0.15)))
+    )
+    (fp_text user "GND" (at -12.8 -19.05 45) (layer "F.SilkS")
+        (effects (font (size 0.8 0.8) (thickness 0.15)))
+    )
+    (fp_text user "GND" (at 12.8 19.05 45) (layer "F.SilkS")
+        (effects (font (size 0.8 0.8) (thickness 0.15)))
+    )
+    (fp_text user "GP12" (at -13.2 13.97 45) (layer "F.SilkS")
+        (effects (font (size 0.8 0.8) (thickness 0.15)))
+    )
+    (fp_text user "GP15" (at -13.054 24.13 45) (layer "F.SilkS")
+        (effects (font (size 0.8 0.8) (thickness 0.15)))
+    )
+    (fp_text user "GP26" (at 13.054 -1.27 45) (layer "F.SilkS")
+        (effects (font (size 0.8 0.8) (thickness 0.15)))
+    )
+    (fp_text user "AGND" (at 13.054 -6.35 45) (layer "F.SilkS")
+        (effects (font (size 0.8 0.8) (thickness 0.15)))
+    )
+    (fp_text user "GND" (at 12.8 -19.05 45) (layer "F.SilkS")
+        (effects (font (size 0.8 0.8) (thickness 0.15)))
+    )
+    (fp_text user "GP20" (at 13.054 11.43 45) (layer "F.SilkS")
+        (effects (font (size 0.8 0.8) (thickness 0.15)))
+    )
+    (fp_text user "GP2" (at -12.9 -16.51 45) (layer "F.SilkS")
+        (effects (font (size 0.8 0.8) (thickness 0.15)))
+    )
+    (fp_text user "GP8" (at -12.8 1.27 45) (layer "F.SilkS")
+        (effects (font (size 0.8 0.8) (thickness 0.15)))
+    )
+    (fp_text user "GP9" (at -12.8 3.81 45) (layer "F.SilkS")
+        (effects (font (size 0.8 0.8) (thickness 0.15)))
+    )
+    (fp_text user "GP7" (at -12.7 -1.3 45) (layer "F.SilkS")
+        (effects (font (size 0.8 0.8) (thickness 0.15)))
+    )
+    (fp_text user "GP6" (at -12.8 -3.81 45) (layer "F.SilkS")
+        (effects (font (size 0.8 0.8) (thickness 0.15)))
+    )
+    (fp_text user "ADC_VREF" (at 14 -12.5 45) (layer "F.SilkS")
+        (effects (font (size 0.8 0.8) (thickness 0.15)))
+    )
+    (fp_text user "GP17" (at 13.054 21.59 45) (layer "F.SilkS")
+        (effects (font (size 0.8 0.8) (thickness 0.15)))
+    )
+    (fp_text user "GP5" (at -12.8 -8.89 45) (layer "F.SilkS")
+        (effects (font (size 0.8 0.8) (thickness 0.15)))
+    )
+    (fp_text user "GP22" (at 13.054 3.81 45) (layer "F.SilkS")
+        (effects (font (size 0.8 0.8) (thickness 0.15)))
+    )
+    (fp_text user "GP16" (at 13.054 24.13 45) (layer "F.SilkS")
+        (effects (font (size 0.8 0.8) (thickness 0.15)))
+    )
+    (fp_text user "GND" (at -12.8 -6.35 45) (layer "F.SilkS")
+        (effects (font (size 0.8 0.8) (thickness 0.15)))
+    )
+    (fp_text user "GP27" (at 13.054 -3.8 45) (layer "F.SilkS")
+        (effects (font (size 0.8 0.8) (thickness 0.15)))
+    )
+    (fp_text user "GP19" (at 13.054 13.97 45) (layer "F.SilkS")
+        (effects (font (size 0.8 0.8) (thickness 0.15)))
+    )
+    (fp_text user "GP3" (at -12.8 -13.97 45) (layer "F.SilkS")
+        (effects (font (size 0.8 0.8) (thickness 0.15)))
+    )
+    (fp_text user "GP14" (at -13.1 21.59 45) (layer "F.SilkS")
+        (effects (font (size 0.8 0.8) (thickness 0.15)))
+    )
+    (fp_text user "GP21" (at 13.054 8.9 45) (layer "F.SilkS")
+        (effects (font (size 0.8 0.8) (thickness 0.15)))
+    )
+    (fp_text user "VBUS" (at 13.3 -24.2 45) (layer "F.SilkS")
+        (effects (font (size 0.8 0.8) (thickness 0.15)))
+    )
+    (fp_text user "GP0" (at -12.8 -24.13 45) (layer "F.SilkS")
+        (effects (font (size 0.8 0.8) (thickness 0.15)))
+    )
+    (fp_text user "GP18" (at 13.054 16.51 45) (layer "F.SilkS")
+        (effects (font (size 0.8 0.8) (thickness 0.15)))
+    )
+    (fp_text user "RUN" (at 13 1.27 45) (layer "F.SilkS")
+        (effects (font (size 0.8 0.8) (thickness 0.15)))
+    )
+    (fp_text user "3V3_EN" (at 13.7 -17.2 45) (layer "F.SilkS")
+        (effects (font (size 0.8 0.8) (thickness 0.15)))
+    )
+    (fp_text user "GP11" (at -13.2 11.43 45) (layer "F.SilkS")
+        (effects (font (size 0.8 0.8) (thickness 0.15)))
+    )
+    (fp_text user "GP28" (at 13.054 -9.144 45) (layer "F.SilkS")
+        (effects (font (size 0.8 0.8) (thickness 0.15)))
+    )
+    (fp_text user "SWCLK" (at -5.7 26.2) (layer "F.SilkS")
+        (effects (font (size 0.8 0.8) (thickness 0.15)))
+    )
+    (fp_text user "GND" (at -12.8 6.35 45) (layer "F.SilkS")
+        (effects (font (size 0.8 0.8) (thickness 0.15)))
+    )
+    (fp_text user "SWDIO" (at 5.6 26.2) (layer "F.SilkS")
+        (effects (font (size 0.8 0.8) (thickness 0.15)))
+    )
+    (fp_text user "Copper Keepouts shown on Dwgs layer" (at 0.1 -30.2) (layer "Cmts.User")
+        (effects (font (size 1 1) (thickness 0.15)))
+    )
+    (fp_text user "${REFERENCE}" (at 0 0 180) (layer "F.Fab")
         (effects (font (size 1 1) (thickness 0.15)))
     )
@@
       (stroke (width 0.12) (type solid)) (layer "F.SilkS"))
     (fp_line (start -3.7 25.5) (end -10.5 25.5)
-      (stroke (width 0.12) (type solid)) (layer "F.SilkS"))
-    (fp_line (start -1.5 25.5) (end -1.1 25.5)
-      (stroke (width 0.12) (type solid)) (layer "F.SilkS"))
-    (fp_line (start 1.1 25.5) (end 1.5 25.5)
       (stroke (width 0.12) (type solid)) (layer "F.SilkS"))
     (fp_line (start 10.5 -25.5) (end 10.5 -25.2)
@@
         (effects (font (size 1 1) (thickness 0.15)))
     )
-    (fp_text value "33k" (at 0.254 0) (layer "F.Fab")
-        (effects (font (size 1 1) (thickness 0.15)))
-    )
+    (fp_text value "27k" (at 0.254 0) (layer "F.Fab")
+        (effects (font (size 1 1) (thickness 0.15)))
+    )

Commit message: Modif of voice board smd and Cleanup
Parts:
- removed J1: ES, SYNTHFILLE:DIP-16_AS
- added J3: Conn_02x09_Counter_Clockwise, AS3397_proto_SMS:DIP-18_AS, F.Cu at (48.3, 47.2)
- R16, R17: value 100k -> 50k
- U1, U3, U5, U7: value MCP6002 -> TS922
- U4: value MCP6002 -> TL072
- moved C33 36.1 mm to (54.3, 58.2), turned to 0 degrees
- moved C30 34.8 mm to (56.9, 141.4), turned to 0 degrees
- moved AS1 33.0 mm to (90.1, 72.5)
- moved C1 33.0 mm to (75.8, 139.2)
- moved C10 33.0 mm to (78.7, 75.5)
- moved C11 33.0 mm to (77.3, 60.9)
- moved C12 33.0 mm to (75.8, 131.0)
- moved C13 33.0 mm to (57.5, 71.6)
- moved C14 33.0 mm to (71.2, 69.1)
- moved C15 33.0 mm to (63.3, 97.2)
- moved C18 33.0 mm to (64.7, 65.5)
- moved C19 33.0 mm to (64.7, 75.2)
- moved C26 33.0 mm to (69.2, 124.4)
- moved C27 33.0 mm to (75.8, 115.3)
- moved C35 33.0 mm to (68.1, 103.6)
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Routing:
- net OUT_R: track 43.8 -> 109.7 mm
- net OUT_L: track 73.5 -> 138.7 mm
- net Net-(U1A-+): track 100.5 -> 63.7 mm, vias 0 -> 2
- net +5V: track 322.3 -> 310.5 mm, vias 7 -> 8
- net I2C_SDA: track 147.7 -> 152.8 mm, vias 2 -> 1
- net I2C_SCK: track 146.4 -> 151.1 mm, vias 2 -> 1
- net +12V: track 172.2 -> 169.6 mm
- net GND: track 748.8 -> 750.6 mm
- net -5V: track 312.1 -> 313.2 mm
- added copper zone on F.Cu, net GND
- removed copper zone on F.Cu, net (none)
Other:
- board size 71.1 x 104.1 mm -> 70.5 x 100.2 mm
