File: hardware/conductor/AS3397-Conductor.kicad_pcb (KiCad board)
At the start: 2 copper layers, 97.3 x 97.8 mm, 49 parts, among them J1 Micro_SD_Card, J10 Conn_FX_2, J11 I2C controller, J12 Conn_01x03_Socket_AudioOUT, J13 Voice connector, J14 Conn_01x02_Socket, J15 I2C controller, J16 Conn_01x06_Socket_SPI, J17 Conn_01x03_Socket, J18 Conn_01x03_Socket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

Commit message: Modif of voice board smd and Cleanup
Parts:
- removed R23, R25: 10K, Resistor_SMD:R_1206_3216Metric_Pad1.30x1.75mm_HandSolder
- added C8: 100n, Capacitor_SMD:C_1206_3216Metric_Pad1.33x1.80mm_HandSolder, F.Cu at (195.7, 108.4)
- added C9: 100n, Capacitor_SMD:C_1206_3216Metric_Pad1.33x1.80mm_HandSolder, F.Cu at (195.8, 100.5)
- added D4: SK6812, LED_SMD:LED_SK6812_PLCC4_5.0x5.0mm_P3.2mm, F.Cu at (189.3, 108.3)
- added D5: SK6812, LED_SMD:LED_SK6812_PLCC4_5.0x5.0mm_P3.2mm, F.Cu at (189.3, 97.1)
- added J19: Conn_Voice, Connector_PinHeader_2.54mm:PinHeader_2x05_P2.54mm_Vertical, F.Cu at (110.6, 123.9)
- added J20: Conn_FX_4, Connector_PinHeader_2.54mm:PinHeader_2x05_P2.54mm_Vertical, F.Cu at (131.4, 114.1)
- added REF**: OSHW-Logo_5.7x6mm_Copper, Symbol:OSHW-Logo_5.7x6mm_Copper, F.Cu at (153.5, 113.7)
- J13: value Voice connector -> Conn_FX_3; footprint Connector_JST:JST_EH_B9B-EH-A_1x09_P2.50mm_Vertical -> Connector_PinHeader_2.54mm:PinHeader_2x05_P2.54mm_Vertical
- moved R28 47.5 mm to (134.7, 150.9), turned to -90 degrees
- moved R27 43.9 mm to (131.4, 151.0), turned to 90 degrees
- moved J13 17.7 mm to (131.3, 104.9)
- moved J9 3.00 mm to (131.3, 95.7)
- moved J10 2.92 mm to (131.3, 86.6)
- moved J3 0.77 mm to (139.6, 107.6)
Connections:
- C6 pad 1: Net-(U3D--) -> Wet_right
- C7 pad 1: Net-(U3A--) -> Wet_left
- J13 pad 1: audio_analog_left -> Dry_left
- J13 pad 2: audio_analog_right -> I2C_CTRL_SDL
- J13 pad 3: I2C_voices_SDL -> Wet_left
- J13 pad 4: I2C_voices_SDA -> I2C_CTRL_SDA
- J13 pad 5: +12V -> Dry_right
- J13 pad 6: GND -> -5V
- J13 pad 7: +5V -> Wet_right
- J13 pad 8: +3.3V -> +12V
- J13 pad 9: -5V -> GND
- R21 pad 1: Net-(U3A--) -> Wet_left
- R22 pad 2: Net-(U3A--) -> Wet_left
- R24 pad 2: Net-(U3D--) -> Wet_right
- R26 pad 1: Net-(U3D--) -> Wet_right
- U3 pad 13: Net-(U3D--) -> Wet_right
- U3 pad 2: Net-(U3A--) -> Wet_left
Routing:
- net Wet_right: track 43.8 -> 82.6 mm
- net +12V: track 83.9 -> 121.3 mm, vias 1 -> 2
- net Wet_left: track 58.1 -> 89.7 mm
- net I2C_CTRL_SDL: track 56.1 -> 86.3 mm
- net audio_analog_right: track 40.6 -> 70.3 mm, vias 0 -> 1
- net -5V: track 140.2 -> 163.8 mm, vias 4 -> 1
- net +5V: track 295.5 -> 318.8 mm, vias 1 -> 3
- net Net-(U3A--): track 22.9 -> 0.00 mm
- net audio_analog_left: track 41.1 -> 62.6 mm
- net Net-(U3D--): track 19.9 -> 0.00 mm
- net I2C_voices_SDL: track 103.9 -> 85.8 mm, vias 2 -> 1
- net I2C_CTRL_SDA: track 86.4 -> 101.4 mm, vias 2 -> 1
- net I2C_voices_SDA: track 96.0 -> 82.0 mm, vias 2 -> 0
- net Dry_left: track 49.8 -> 60.3 mm
- net Dry_right: track 59.1 -> 49.6 mm, vias 1 -> 0
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Other:
- outline, holes or cut-outs redrawn
- board text added: "5V 12V -5V SDA SDL"
- board text added: "Conductor"
- board text added: "Conductor v1.0"
- board text added: "GND -5V 3.3V +5V GND"
- board text added: "GND WR DR WL DL"
- board text added: "L R SCL SDA 12V"
- board text added: "TX1 RX1"
- board text removed: "L R SCL SDA 12 GND +5 ADD -5"
