File: hardware/voice/mono - through-hole/AS3397_proto_DIP.kicad_pcb (KiCad board)
At the start: 2 copper layers, 167.6 x 97.5 mm, 142 parts, among them J1 +15V, J2 MIDI IN, J3 OUTPUT, J4 I2C, Q2 BS170, Q3 BS170, Q4 BS170, Q5 BS170, U1 TC7662, U10 LM7805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

Commit message: Voice firmware  big improvement and through hole board fixes
Connections:
- U5 pad 8: -5V -> +5V
Routing:
- net -5V: track 350.9 -> 345.9 mm
- net +5V: track 417.1 -> 419.9 mm

Commit message: Conductor board new version
Parts:
- C27: footprint Capacitor_THT:C_Rect_L7.0mm_W2.0mm_P5.00mm -> Capacitor_THT:C_Rect_L7.0mm_W3.5mm_P5.00mm
- R23, R24: value 100k -> 50K
- U11, U4, U8, U9: value MCP6002 -> TS922
- moved C27 0.81 mm to (173.9, 111.3)
Changed lines of the file:
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@@
 			)
 		)
-		(property "Value" "100k"
+		(property "Value" "50K"
 			(at 3.81 0 90)
 			(layer "F.SilkS")
@@
 			)
 		)
-		(property "Value" "MCP6002"
+		(property "Value" "TS922"
 			(at 5.334 3.81 90)
 			(layer "F.SilkS")
@@
 			)
 		)
-		(property "Value" "MCP6002"
+		(property "Value" "TS922"
 			(at 5.334 3.556 90)
 			(layer "F.SilkS")
@@
 		)
 	)
-	(footprint "Capacitor_THT:C_Rect_L7.0mm_W2.0mm_P5.00mm"
+	(footprint "Capacitor_THT:C_Rect_L7.0mm_W3.5mm_P5.00mm"
 		(layer "F.Cu")
-		(at 173.99 110.49 180)
-		(descr "C, Rect series, Radial, pin pitch=5.00mm, , length*width=7*2mm^2, Capacitor")
-		(tags "C Rect series Radial pin pitch 5.00mm  length 7mm width 2mm Capacitor")
+		(at 173.9354 111.3028 180)
+		(descr "C, Rect series, Radial, pin pitch=5.00mm, , length*width=7*3.5mm^2, Capacitor")
+		(tags "C Rect series Radial pin pitch 5.00mm  length 7mm width 3.5mm Capacitor")
 		(property "Reference" "C27"
-			(at 2.5 -2.25 0)
+			(at 2.5 -3 180)
 			(layer "F.SilkS")
 			(effects
@@
 		)
 		(property "Value" "1uF"
-			(at 2.54 0 0)
-			(layer "F.SilkS")
+			(at 2.5 3 180)
+			(layer "F.Fab")
 			(effects
 				(font
@@
 		(property "Datasheet" ""
 			(at 0 0 180)
+			(unlocked yes)
 			(layer "F.Fab")
 			(hide yes)
@@
 		(property "Description" ""
 			(at 0 0 180)
+			(unlocked yes)
 			(layer "F.Fab")
 			(hide yes)
@@
 		(attr through_hole)
 		(fp_line
-			(start 6.12 -1.12)
-			(end 6.12 1.12)
+			(start 6.12 -1.87)
+			(end 6.12 1.87)
 			(stroke
 				(width 0.12)
@@
 		)
 		(fp_line
-			(start -1.12 1.12)
-			(end 6.12 1.12)
+			(start -1.12 1.87)
+			(end 6.12 1.87)
 			(stroke
 				(width 0.12)
@@
 		)
 		(fp_line
-			(start -1.12 -1.12)
-			(end 6.12 -1.12)
+			(start -1.12 -1.87)
+			(end 6.12 -1.87)
 			(stroke
 				(width 0.12)
@@
 		)
 		(fp_line
-			(start -1.12 -1.12)
-			(end -1.12 1.12)
+			(start -1.12 -1.87)
+			(end -1.12 1.87)
 			(stroke
 				(width 0.12)
@@
 		)
 		(fp_line
-			(start 6.25 1.25)
-			(end 6.25 -1.25)
+			(start 6.25 2)
+			(end 6.25 -2)
 			(stroke
 				(width 0.05)
@@
 		)
 		(fp_line
-			(start 6.25 -1.25)
-			(end -1.25 -1.25)
+			(start 6.25 -2)
+			(end -1.25 -2)
 			(stroke
 				(width 0.05)
@@
 		)
 		(fp_line
-			(start -1.25 1.25)
-			(end 6.25 1.25)
+			(start -1.25 2)
+			(end 6.25 2)
 			(stroke
 				(width 0.05)
@@
 		)
 		(fp_line
-			(start -1.25 -1.25)
-			(end -1.25 1.25)
+			(start -1.25 -2)
+			(end -1.25 2)
 			(stroke
 				(width 0.05)
@@
 		)
 		(fp_line
-			(start 6 1)
-			(end 6 -1)
+			(start 6 1.75)
+			(end 6 -1.75)
 			(stroke
 				(width 0.1)
@@
 		)
 		(fp_line
-			(start 6 -1)
-			(end -1 -1)
+			(start 6 -1.75)
+			(end -1 -1.75)
 			(stroke
 				(width 0.1)
@@
 		)
 		(fp_line
-			(start -1 1)
-			(end 6 1)
+			(start -1 1.75)
+			(end 6 1.75)
 			(stroke
 				(width 0.1)
@@
 		)
 		(fp_line
-			(start -1 -1)
-			(end -1 1)
+			(start -1 -1.75)
+			(end -1 1.75)
 			(stroke
 				(width 0.1)
@@
 			(layer "F.Fab")
 		)
+		(fp_text user "${REFERENCE}"
+			(at 2.5 0 180)
+			(layer "F.Fab")
+			(effects
+				(font
+					(size 1 1)
+					(thickness 0.15)
+				)
+			)
+		)
 		(pad "1" thru_hole circle
 			(at 0 0 180)
@@
 		)
 		(embedded_fonts no)
-		(model "${KICAD6_3DMODEL_DIR}/Capacitor_THT.3dshapes/C_Rect_L7.0mm_W2.0mm_P5.00mm.wrl"
+		(model "${KICAD9_3DMODEL_DIR}/Capacitor_THT.3dshapes/C_Rect_L7.0mm_W3.5mm_P5.00mm.wrl"
 			(offset
 				(xyz 0 0 0)
@@
 			)
 		)
-		(property "Value" "MCP6002"
+		(property "Value" "TS922"
 			(at 2.286 4.064 90)
 			(layer "F.SilkS")
@@
 			)
 		)
-		(property "Value" "MCP6002"
+		(property "Value" "TS922"
 			(at 3.81 9.95 0)
 			(layer "F.SilkS")
@@
 			)
 		)
-		(property "Value" "100k"
+		(property "Value" "50K"
 			(at 3.715 -0.015 90)
 			(layer "F.SilkS")
@@
 	)
 	(segment
-		(start 183.515 105.41)
-		(end 184.4675 104.4575)
-		(width 0.25)
-		(layer "B.Cu")
-		(net 13)
-	)
-	(segment
-		(start 169.545 117.4825)
-		(end 172.0775 117.4825)
+		(start 189.23 97.775)
+		(end 188.976 97.775)
 		(width 0.25)
 		(layer "B.Cu")
@@
 	)
 	(segment
-		(start 184.4675 104.4575)
-		(end 184.4675 98.7425)
+		(start 174.625 105.41)
+		(end 183.515 105.41)
 		(width 0.25)
 		(layer "B.Cu")
@@
 	)
 	(segment
-		(start 168.925 118.1025)
-		(end 169.545 117.4825)
+		(start 185.435 97.775)
+		(end 189.738 97.775)
 		(width 0.25)
 		(layer "B.Cu")
@@
 	)
 	(segment
-		(start 189.23 97.775)
+		(start 188.976 92.964)
 		(end 188.976 97.775)
 		(width 0.25)
@@
 	)
 	(segment
-		(start 188.976 92.964)
-		(end 188.976 97.775)
+		(start 169.545 117.4825)
+		(end 172.0775 117.4825)
 		(width 0.25)
 		(layer "B.Cu")
@@
 	)
 	(segment
-		(start 184.4675 98.7425)
-		(end 185.435 97.775)
+		(start 172.0775 117.4825)
+		(end 172.6438 116.9162)
 		(width 0.25)
 		(layer "B.Cu")
@@
 	)
 	(segment
-		(start 172.785 107.38)
-		(end 172.72 107.315)
+		(start 183.515 105.41)
+		(end 184.4675 104.4575)
 		(width 0.25)
 		(layer "B.Cu")
@@
 	)
 	(segment
-		(start 172.72 107.315)
-		(end 174.625 105.41)
+		(start 184.4675 104.4575)
+		(end 184.4675 98.7425)
 		(width 0.25)
 		(layer "B.Cu")
@@
 	)
 	(segment
-		(start 172.785 116.775)
-		(end 172.785 107.38)
+		(start 189.738 97.775)
+		(end 189.23 97.775)
 		(width 0.25)
 		(layer "B.Cu")
@@
 	)
 	(segment
-		(start 174.625 105.41)
-		(end 183.515 105.41)
+		(start 168.925 119.38)
+		(end 168.925 118.1025)
 		(width 0.25)
 		(layer "B.Cu")
@@
 	(segment
 		(start 168.925 119.38)
-		(end 168.925 118.1025)
+		(end 166.37 119.38)
 		(width 0.25)
 		(layer "B.Cu")
@@
 	)
 	(segment
-		(start 189.738 97.775)
-		(end 189.23 97.775)
+		(start 172.6438 107.3912)
+		(end 174.625 105.41)
 		(width 0.25)
 		(layer "B.Cu")
@@
 	)
 	(segment
-		(start 189.738 97.775)
-		(end 185.435 97.775)
+		(start 168.925 118.1025)
+		(end 169.545 117.4825)
 		(width 0.25)
 		(layer "B.Cu")
@@
 	)
 	(segment
-		(start 168.925 119.38)
-		(end 166.37 119.38)
+		(start 172.6438 116.9162)
+		(end 172.6438 107.3912)
 		(width 0.25)
 		(layer "B.Cu")
@@
 	)
 	(segment
-		(start 172.0775 117.4825)
-		(end 172.785 116.775)
+		(start 184.4675 98.7425)
+		(end 185.435 97.775)
 		(width 0.25)
 		(layer "B.Cu")
@@
 	)
 	(segment
-		(start 168.91 113.029302)
-		(end 152.400698 113.029302)
+		(start 152.400698 113.029302)
+		(end 150.114 115.316)
 		(width 0.25)
 		(layer "B.Cu")
@@
 	)
 	(segment
-		(start 191.77 85.075)
-		(end 194.325 85.075)
+		(start 150.114 115.316)
+		(end 150.114 122.936)
 		(width 0.25)
 		(layer "B.Cu")
@@
 	)
 	(segment
-		(start 170.179302 106.045698)
-		(end 170.179302 111.76)
+		(start 172.72 103.505)
+		(end 170.179302 106.045698)
 		(width 0.25)
 		(layer "B.Cu")
@@
 	)
 	(segment
-		(start 150.114 115.316)
-		(end 150.114 122.936)
+		(start 170.179302 106.045698)
+		(end 170.179302 112.065498)
 		(width 0.25)
 		(layer "B.Cu")
@@
 	)
 	(segment
-		(start 172.72 91.44)
-		(end 172.72 103.505)
+		(start 191.77 85.075)
+		(end 194.325 85.075)
 		(width 0.25)
 		(layer "B.Cu")
@@
 	)
 	(segment
-		(start 170.179302 111.76)
-		(end 168.91 113.029302)
+		(start 169.215498 113.029302)
+		(end 152.400698 113.029302)
 		(width 0.25)
 		(layer "B.Cu")
@@
 	)
 	(segment
-		(start 172.72 103.505)
-		(end 170.179302 106.045698)
+		(start 172.72 91.44)
+		(end 172.72 103.505)
 		(width 0.25)
 		(layer "B.Cu")
@@
 	)
 	(segment
-		(start 152.400698 113.029302)
-		(end 150.114 115.316)
+		(start 170.179302 112.065498)
+		(end 169.215498 113.029302)
 		(width 0.25)
 		(layer "B.Cu")
@@
 	)
 	(segment
+		(start 168.1226 110.49)
+		(end 163.83 110.49)
+		(width 0.25)
+		(layer "B.Cu")
+		(net 20)
+	)
+	(segment
 		(start 100.195 90.035)
 		(end 104.775 94.615)
@@
 	)
 	(segment
-		(start 163.83 110.49)
-		(end 168.99 110.49)
+		(start 168.9354 111.3028)
+		(end 168.1226 110.49)
 		(width 0.25)
 		(layer "B.Cu")
@@
 	)
 	(segment
-		(start 177.8 110.49)
-		(end 173.99 110.49)
+		(start 176.9872 111.3028)
+		(end 177.8 110.49)
+		(width 0.25)
+		(layer "B.Cu")
+		(net 115)
+	)
+	(segment
+		(start 173.9354 111.3028)
+		(end 176.9872 111.3028)
 		(width 0.25)
 		(layer "B.Cu")
