File: hardware/voice/mono - through-hole/AS3397_proto_DIP.kicad_sch (KiCad schematic)
At the start: 142 parts, among them J1 +15V, J2 MIDI IN, J3 OUTPUT, J4 I2C, Q2 BS170, Q3 BS170, Q4 BS170, Q5 BS170, U1 TC7662, U10 LM7805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

Commit message: Voice firmware  big improvement and through hole board fixes
Connections:
- net +5V: now also U5.8 (VCC)
- net -5V: no longer U5.8 (VCC)

Commit message: Conductor board new version
Parts:
- R23, R24: value 100k -> 50K
- U11, U4, U8, U9: value MCP6002 -> TS922
Other:
- note added: "Compatible op-amp TCL2262 or TLV9102 TLV2372"
Changed lines of the file:
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@@
 		)
 	)
+	(text "Compatible op-amp\nTCL2262 or TLV9102 \nTLV2372\n"
+		(exclude_from_sim no)
+		(at 417.322 370.84 0)
+		(effects
+			(font
+				(size 1.27 1.27)
+			)
+			(justify left)
+		)
+	)
 	(text "Registers change"
 		(exclude_from_sim no)
@@
 		)
 	)
+	(text "Compatible op-amp\nTCL2262 or TLV9102 \nTLV2372\n"
+		(exclude_from_sim no)
+		(at 113.03 244.094 0)
+		(effects
+			(font
+				(size 1.27 1.27)
+			)
+			(justify left)
+		)
+	)
+	(text "Compatible op-amp\nTCL2262 or TLV9102 \nTLV2372\n"
+		(exclude_from_sim no)
+		(at 276.098 309.118 0)
+		(effects
+			(font
+				(size 1.27 1.27)
+			)
+			(justify left)
+		)
+	)
 	(text "0V to 5V\n"
 		(exclude_from_sim no)
@@
 		)
 	)
+	(text "Compatible op-amp\nTCL2262 or TLV9102 \nTLV2372\n"
+		(exclude_from_sim no)
+		(at 265.43 325.12 0)
+		(effects
+			(font
+				(size 1.27 1.27)
+			)
+			(justify left)
+		)
+	)
 	(text "level shifter\nPWM low-pass filtering"
 		(exclude_from_sim no)
@@
 		)
 	)
+	(text "Compatible op-amp\nTCL2262 or TLV9102 \nTLV2372\n"
+		(exclude_from_sim no)
+		(at 245.364 244.094 0)
+		(effects
+			(font
+				(size 1.27 1.27)
+			)
+			(justify left)
+		)
+	)
 	(text "-0.5V to 5V\n"
 		(exclude_from_sim no)
@@
 			)
 		)
-		(property "Value" "MCP6002"
+		(property "Value" "TS922"
 			(at 308.102 278.13 0)
 			(effects
@@
 			)
 		)
-		(property "Value" "MCP6002"
+		(property "Value" "TS922"
 			(at 441.452 287.528 0)
 			(effects
@@
 		(on_board yes)
 		(dnp no)
-		(fields_autoplaced yes)
 		(property "Reference" "R24"
-			(at 270.51 109.22 90)
+			(at 269.748 113.03 90)
 			(effects
 				(font
@@
 			)
 		)
-		(property "Value" "100k"
-			(at 270.51 111.76 90)
+		(property "Value" "50K"
+			(at 274.828 113.03 90)
 			(effects
 				(font
@@
 		(fields_autoplaced yes)
 		(property "Reference" "U8"
-			(at 194.31 252.73 0)
+			(at 194.31 251.46 0)
 			(effects
 				(font
@@
 			)
 		)
-		(property "Value" "MCP6002"
-			(at 194.31 255.27 0)
+		(property "Value" "TS922"
+			(at 194.31 254 0)
 			(effects
 				(font
@@
 		(on_board yes)
 		(dnp no)
-		(fields_autoplaced yes)
 		(property "Reference" "R23"
-			(at 270.51 76.2 90)
+			(at 266.954 80.264 90)
 			(effects
 				(font
@@
 			)
 		)
-		(property "Value" "100k"
-			(at 270.51 78.74 90)
+		(property "Value" "50K"
+			(at 272.034 79.756 90)
 			(effects
 				(font
@@
 		(fields_autoplaced yes)
 		(property "Reference" "U11"
-			(at 96.52 334.01 0)
+			(at 96.52 332.74 0)
 			(effects
 				(font
@@
 			)
 		)
-		(property "Value" "MCP6002"
-			(at 96.52 336.55 0)
+		(property "Value" "TS922"
+			(at 96.52 335.28 0)
 			(effects
 				(font
@@
 			)
 		)
-		(property "Value" "MCP6002"
+		(property "Value" "TS922"
 			(at 378.46 262.89 0)
 			(effects
@@
 			)
 		)
-		(property "Value" "MCP6002"
+		(property "Value" "TS922"
 			(at 139.7 379.73 0)
 			(effects
@@
 			)
 		)
-		(property "Value" "MCP6002"
+		(property "Value" "TS922"
 			(at 497.84 317.5 0)
 			(effects
@@
 			)
 		)
-		(property "Value" "MCP6002"
+		(property "Value" "TS922"
 			(at 234.696 269.748 0)
 			(effects
@@
 		(dnp no)
 		(property "Reference" "U6"
-			(at 271.78 87.63 0)
+			(at 272.542 93.472 0)
 			(effects
 				(font
@@
 		)
 		(property "Value" "TL072"
-			(at 271.78 86.36 0)
+			(at 272.034 86.106 0)
 			(effects
 				(font
@@
 			)
 		)
-		(property "Value" "MCP6002"
+		(property "Value" "TS922"
 			(at 378.46 293.37 0)
 			(effects
@@
 			)
 		)
-		(property "Value" "MCP6002"
+		(property "Value" "TS922"
 			(at 222.25 337.82 0)
 			(effects
@@
 			)
 		)
-		(property "Value" "MCP6002"
+		(property "Value" "TS922"
 			(at 81.28 259.08 0)
 			(effects
@@
 			)
 		)
-		(property "Value" "MCP6002"
+		(property "Value" "TS922"
 			(at 496.57 252.73 0)
 			(effects
